File: project/_psu.kicad_sch (KiCad schematic)
At the start: 39 parts, among them J301 24V, J302 5V, J303 3V3, J304 6V, Q301 MMBT3904, U301 LW6550A23E, U302 JTD6206-3.3V, U303 ME3121AM6G

Commit message: spritting up boards into separate repos
Other:
- title: WormControl-Relay15x5t15-ControlUI -> WormControl-Relay15x5t15-ControlBoard
Changed lines of the file:
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@@
   (paper "A4")
   (title_block
-    (title "WormControl-Relay15x5t15-ControlUI")
-    (date "2024-12-19")
-    (rev "0.1")
+    (title "WormControl-Relay15x5t15-ControlBoard")
+    (date "2026-03-19")
+    (rev "0.4")
     (company "makerspace.lt")
   )
@@
       (effects (font (size 1.27 1.27)) hide)
     )
-    (property "LCSC#" "" (id 4) (at 36.83 62.23 90)
-      (effects (font (size 1.27 1.27)) hide)
-    )
