File: project/_uc.kicad_sch (KiCad schematic)
At the start: 35 parts, among them J401 USB_C_Receptacle_USB2.0, SW401 15mm, SW402 15mm, U401 USBLC6-2SC6, U402 esp32-C3FH4X, U403 XL1050, Y401 40MHz

Commit message: spritting up boards into separate repos
Other:
- title: WormControl-Relay15x5t15-ControlUI -> WormControl-Relay15x5t15-ControlBoard
Changed lines of the file:
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@@
   (paper "A4")
   (title_block
-    (title "WormControl-Relay15x5t15-ControlUI")
-    (date "2024-12-19")
-    (rev "0.1")
+    (title "WormControl-Relay15x5t15-ControlBoard")
+    (date "2026-03-19")
+    (rev "0.4")
     (company "makerspace.lt")
   )

Commit message: part consolidation and QoL improvements
* Using same crystal as in other projects
* Switching to TMP102 as TMP101 is no longer available
* Adding cutouts to make assembly esier
* Making net names more readable
* bumping up version
Parts:
- Y401: footprint Crystal:Crystal_SMD_3225-4Pin_3.2x2.5mm -> -local:Crystal_SMD_2016-4Pin_2.0x1.6mm; lcsc# C19191260 -> C20885029
Changed lines of the file:
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@@
     (title "WormControl-Relay15x5t15-ControlBoard")
     (date "2026-03-19")
-    (rev "0.4")
+    (rev "0.5")
     (company "makerspace.lt")
   )
@@
     (property "Reference" "Y401" (id 0) (at 36.83 101.6 0))
     (property "Value" "40MHz" (id 1) (at 54.61 101.6 0))
-    (property "Footprint" "Crystal:Crystal_SMD_3225-4Pin_3.2x2.5mm" (id 2) (at 46.99 104.14 0)
-      (effects (font (size 1.27 1.27)) hide)
-    )
-    (property "Datasheet" "https://wmsc.lcsc.com/wmsc/upload/file/pdf/v2/lcsc/2311101855_SST-SCGYS40X00000YLXWPM_C19191260.pdf" (id 3) (at 46.99 104.14 0)
+    (property "Footprint" "-local:Crystal_SMD_2016-4Pin_2.0x1.6mm" (id 2) (at 46.99 104.14 0)
+      (effects (font (size 1.27 1.27)) hide)
+    )
+    (property "Datasheet" "https://www.lcsc.com/datasheet/C20885029.pdf" (id 3) (at 46.99 104.14 0)
       (effects (font (size 1.27 1.27)) hide)
     )
@@
       (effects (font (size 1.27 1.27)) hide)
     )
-    (property "lcsc#" "C19191260" (id 5) (at 46.99 104.14 0)
-      (effects (font (size 1.27 1.27)) hide)
-    )
+    (property "lcsc#" "C20885029" (id 5) (at 46.99 104.14 0)
+      (effects (font (size 1.27 1.27)) hide)
+    )
